Commit message: Setting wheel radius to 0.01

File: urdf/cmexa/cmexa_properties.urdf.xacro (robot description, xacro)
@@ -11,6 +11,6 @@
   <xacro:property name="wheel_vertical_offset" value="0.01" />
   <xacro:property name="footprint_vertical_offset" value="0.025" />
-  <xacro:property name="wheel_radius" value="0.050" />
-  <xacro:property name="wheel_width" value="0.050" />
+  <xacro:property name="wheel_radius" value="0.001" />
+  <xacro:property name="wheel_width" value="0.001" />
   <xacro:property name="chassis_length" value="0.500" />
   <xacro:property name="chassis_width" value="0.350" />
