Commit message: Backporting cmexaiii changes to cmexa (base_link to chassis and joint corrections)

File: urdf/cmexa/cmexa_description.urdf.xacro (robot description, xacro)
@@ -6,34 +6,41 @@
   <xacro:property name="z_offset" value="-${chassis_height/2}" /> <!-- Space btw top of beam and the each joint -->
   <xacro:property name="wheel_mass" value="0.3"/>
-  <!-- Base Link -->
-  <link name="${prefix}base_link">
-    <collision>
-      <origin xyz="0 0 0" rpy="0 0 0"/>
+    <!-- Base Link -->
+  <link name="${prefix}base_link"></link>
+  <joint name="base_link_joint" type="fixed">
+    <origin xyz="0 0 ${wheel_radius/2}" rpy="0 0 0" />
+    <parent link="${prefix}base_link"/>
+    <child link="${prefix}chassis_link" />
+  </joint>
+  <link name="${prefix}chassis_link">
+    <visual>
+      <origin xyz="${chassis_length/2} ${-chassis_width/2} 0" rpy="0 0 ${PI/2}" />
       <geometry>
-        <!--<box size="${chassis_width} ${chassis_length} ${chassis_height}"/>-->
         <mesh filename="package://cmeresearch_description/meshes/cmexa/cmexa-base.stl" scale="0.001 0.001 0.001"/>
       </geometry>
+      <material name="dark_grey" />
+    </visual>
+    <collision>
+      <origin xyz="${chassis_length/2} ${chassis_width/2} ${chassis_height/2}"/>
+      <geometry>
+        <box size="${chassis_length} ${chassis_width} ${chassis_height}"/>
+      </geometry>
     </collision>
-    <visual>
-      <origin xyz="0 0 ${chassis_height/2}" rpy="0 0 0"/>
-      <geometry>
-        <box size="${chassis_width} ${chassis_length} ${chassis_height}"/>
-      </geometry>
-      <material name="orange"/>
-    </visual>
     <inertial>
-      <origin xyz="0 0 0" rpy="0 0 0"/>
-      <mass value="${chassis_mass}"/>
+      <!-- Center of mass -->
+      <origin xyz="0.012  0.002 0.067" rpy="0 0 0"/>
+      <mass value="16.523"/>
+      <!-- Moments of inertia: ( chassis without wheels ) -->
       <inertia
-        ixx="${chassis_mass / 12.0 * (chassis_length*chassis_length + chassis_height*chassis_height)}" ixy="0.0" ixz="0.0"
-        iyy="${chassis_mass / 12.0 * (chassis_height*chassis_height + chassis_width*chassis_width)}" iyz="0.0"
-        izz="${chassis_mass / 12.0 * (chassis_width*chassis_width + chassis_length*chassis_length)}"/>
+        ixx="0.3136" ixy="-0.0008" ixz="0.0164"
+        iyy="0.3922" iyz="-0.0009"
+        izz="0.4485"/>
       </inertial>
-    </link>
+  </link>
     <!-- Front left wheel -->
     <joint name="${prefix}front_left_wheel_joint" type="continuous">
       <parent link="${prefix}base_link"/>
       <child link="${prefix}front_left_wheel"/>
-      <origin xyz="${chassis_width/2} ${chassis_length/2} ${z_offset}" rpy="0 0 0"/>
+      <origin xyz="${wheelbase/2} ${track/2} ${wheel_radius/2}" rpy="0 0 0"/>
       <axis xyz="0 1 0"/>
       <dynamics damping="0.2"/>
@@ -68,5 +75,5 @@
       <parent link="${prefix}base_link"/>
       <child link="${prefix}front_right_wheel"/>
-      <origin xyz="-${chassis_width/2} ${chassis_length/2} ${z_offset}" rpy="0 0 0"/>
+      <origin xyz="${-wheelbase/2} ${track/2} ${wheel_radius/2}" rpy="0 0 0"/>
       <axis xyz="0 1 0"/>
       <dynamics damping="0.2"/>
@@ -101,5 +108,5 @@
       <parent link="${prefix}base_link"/>
       <child link="${prefix}rear_left_wheel"/>
-      <origin xyz="${chassis_width/2} -${chassis_length/2} ${z_offset}" rpy="0 0 0"/>
+      <origin xyz="${wheelbase/2} ${-track/2} ${wheel_radius/2}" rpy="0 0 0"/>
       <axis xyz="0 1 0"/>
       <dynamics damping="0.2"/>
@@ -134,5 +141,5 @@
       <parent link="${prefix}base_link"/>
       <child link="${prefix}rear_right_wheel"/>
-      <origin xyz="-${chassis_width/2} -${chassis_length/2} ${z_offset}" rpy="0 0 0"/>
+      <origin xyz="${-wheelbase/2} ${-track/2} ${wheel_radius/2}" rpy="0 0 0"/>
       <axis xyz="0 1 0"/>
       <dynamics damping="0.2"/>

File: urdf/cmexa/cmexa_properties.urdf.xacro (robot description, xacro)
@@ -10,10 +10,10 @@
   <!-- vertical offset means height -->
   <xacro:property name="wheel_vertical_offset" value="0.01" />
-  <xacro:property name="footprint_vertical_offset" value="0.0" />
-  <xacro:property name="wheel_radius" value="0.05" />
+  <xacro:property name="footprint_vertical_offset" value="0.025" />
+  <xacro:property name="wheel_radius" value="0.050" />
   <xacro:property name="wheel_width" value="0.050" />
-  <xacro:property name="chassis_length" value="0.200" />
-  <xacro:property name="chassis_width" value="0.130" />
-  <xacro:property name="chassis_height" value="0.150" />
+  <xacro:property name="chassis_length" value="0.500" />
+  <xacro:property name="chassis_width" value="0.350" />
+  <xacro:property name="chassis_height" value="0.300" />
   <xacro:property name="chassis_mass" value="0.3" /> <!-- correct this later -->
   <xacro:property name="dummy_inertia" value="1e-09"/>

Commit message: Trying mirrored axis for rear wheels.

File: urdf/cmexa/cmexa_description.urdf.xacro (robot description, xacro)
@@ -104,5 +104,5 @@
     <child link="${prefix}rear_left_wheel"/>
     <origin xyz="${wheelbase/2} ${-track/2} ${wheel_radius/2}" rpy="0 0 0"/>
-    <axis xyz="0 1 0"/>
+    <axis xyz="0 -1 0"/>
     <dynamics damping="0.2"/>
     <limit effort="100" velocity="1.0"/>
@@ -137,5 +137,5 @@
     <child link="${prefix}rear_right_wheel"/>
     <origin xyz="${-wheelbase/2} ${-track/2} ${wheel_radius/2}" rpy="0 0 0"/>
-    <axis xyz="0 1 0"/>
+    <axis xyz="0 -1 0"/>
     <dynamics damping="0.2"/>
     <limit effort="100" velocity="1.0"/>

Commit message: Trying mirrored axis for rear wheels.

File: urdf/cmexa/cmexa_description.urdf.xacro (robot description, xacro)
@@ -104,5 +104,5 @@
     <child link="${prefix}rear_left_wheel"/>
     <origin xyz="${wheelbase/2} ${-track/2} ${wheel_radius/2}" rpy="0 0 0"/>
-    <axis xyz="0 -1 0"/>
+    <axis xyz="0 1 0"/>
     <dynamics damping="0.2"/>
     <limit effort="100" velocity="1.0"/>
@@ -137,5 +137,5 @@
     <child link="${prefix}rear_right_wheel"/>
     <origin xyz="${-wheelbase/2} ${-track/2} ${wheel_radius/2}" rpy="0 0 0"/>
-    <axis xyz="0 -1 0"/>
+    <axis xyz="0 1 0"/>
     <dynamics damping="0.2"/>
     <limit effort="100" velocity="1.0"/>

Commit message: Trying mirrored axis for front wheels.

File: urdf/cmexa/cmexa_description.urdf.xacro (robot description, xacro)
@@ -38,5 +38,5 @@
     <child link="${prefix}front_left_wheel"/>
     <origin xyz="${wheelbase/2} ${track/2} ${wheel_radius/2}" rpy="0 0 0"/>
-    <axis xyz="0 1 0"/>
+    <axis xyz="0 -1 0"/>
     <dynamics damping="0.2"/>
     <limit effort="100" velocity="1.0"/>
@@ -71,5 +71,5 @@
     <child link="${prefix}front_right_wheel"/>
     <origin xyz="${-wheelbase/2} ${track/2} ${wheel_radius/2}" rpy="0 0 0"/>
-    <axis xyz="0 1 0"/>
+    <axis xyz="0 -1 0"/>
     <dynamics damping="0.2"/>
     <limit effort="100" velocity="1.0"/>

Commit message: Trying mirrored axis for front wheels.

File: urdf/cmexa/cmexa_description.urdf.xacro (robot description, xacro)
@@ -38,5 +38,5 @@
     <child link="${prefix}front_left_wheel"/>
     <origin xyz="${wheelbase/2} ${track/2} ${wheel_radius/2}" rpy="0 0 0"/>
-    <axis xyz="0 -1 0"/>
+    <axis xyz="0 1 0"/>
     <dynamics damping="0.2"/>
     <limit effort="100" velocity="1.0"/>
@@ -71,5 +71,5 @@
     <child link="${prefix}front_right_wheel"/>
     <origin xyz="${-wheelbase/2} ${track/2} ${wheel_radius/2}" rpy="0 0 0"/>
-    <axis xyz="0 -1 0"/>
+    <axis xyz="0 1 0"/>
     <dynamics damping="0.2"/>
     <limit effort="100" velocity="1.0"/>

Commit message: Trying mirrored axis for front wheels.

File: urdf/cmexa/cmexa_description.urdf.xacro (robot description, xacro)
@@ -33,4 +33,28 @@
       </inertial>
   </link>
+   <!-- front left wheel Link -->
+   <link name="${prefix}front_left_wheel">
+     <collision>
+       <origin xyz="0 0 0" rpy="0 0 0"/>
+       <geometry>
+         <cylinder length="${wheel_width}" radius="${wheel_radius}"/>
+       </geometry>
+     </collision>
+     <visual>
+       <origin xyz="0 0 0" rpy="0 0 0"/>
+       <geometry>
+         <cylinder length="${wheel_width}" radius="${wheel_radius}"/>
+       </geometry>
+       <material name="black"/>
+     </visual>
+     <inertial>
+       <origin xyz="0 0 0" rpy="0 0 0"/>
+       <mass value="${wheel_mass}"/>
+       <inertia
+               ixx="${wheel_mass / 12.0 * (3*wheel_radius*wheel_radius + wheel_width*wheel_width)}" ixy="0.0" ixz="0.0"
+               iyy="${wheel_mass / 12.0 * (3*wheel_radius*wheel_radius + wheel_width*wheel_width)}" iyz="0.0"
+               izz="${wheel_mass / 2.0 * wheel_radius*wheel_radius}"/>
+     </inertial>
+   </link>
     <!-- Front left wheel -->
   <joint name="${prefix}front_left_wheel_joint" type="continuous">
@@ -42,28 +66,4 @@
     <limit effort="100" velocity="1.0"/>
   </joint>
-  <!-- front left wheel Link -->
-  <link name="${prefix}front_left_wheel">
-    <collision>
-      <origin xyz="0 0 0" rpy="${PI/2} 0 0"/>
-      <geometry>
-        <cylinder length="${wheel_width}" radius="${wheel_radius}"/>
-      </geometry>
-    </collision>
-    <visual>
-      <origin xyz="0 0 0" rpy="${PI/2} 0 0"/>
-      <geometry>
-        <cylinder length="${wheel_width}" radius="${wheel_radius}"/>
-      </geometry>
-      <material name="black"/>
-    </visual>
-    <inertial>
-      <origin xyz="0 0 0" rpy="${PI/2} 0 0"/>
-      <mass value="${wheel_mass}"/>
-      <inertia
-              ixx="${wheel_mass / 12.0 * (3*wheel_radius*wheel_radius + wheel_width*wheel_width)}" ixy="0.0" ixz="0.0"
-              iyy="${wheel_mass / 12.0 * (3*wheel_radius*wheel_radius + wheel_width*wheel_width)}" iyz="0.0"
-              izz="${wheel_mass / 2.0 * wheel_radius*wheel_radius}"/>
-    </inertial>
-  </link>
   <!-- Front right wheel -->
   <joint name="${prefix}front_right_wheel_joint" type="continuous">

Commit message: Changing velocity limits on xml.

File: urdf/cmexa/cmexa_description.urdf.xacro (robot description, xacro)
@@ -64,5 +64,5 @@
     <axis xyz="0 1 0"/>
     <dynamics damping="0.2"/>
-    <limit effort="100" velocity="1.0"/>
+    <limit effort="100" velocity="5.0"/>
   </joint>
   <!-- Front right wheel -->
@@ -73,5 +73,5 @@
     <axis xyz="0 1 0"/>
     <dynamics damping="0.2"/>
-    <limit effort="100" velocity="1.0"/>
+    <limit effort="100" velocity="5.0"/>
   </joint>
   <!-- front right wheel Link -->
@@ -106,5 +106,5 @@
     <axis xyz="0 1 0"/>
     <dynamics damping="0.2"/>
-    <limit effort="100" velocity="1.0"/>
+    <limit effort="100" velocity="5.0"/>
   </joint>
   <!-- rear left wheel Link -->
@@ -139,5 +139,5 @@
     <axis xyz="0 1 0"/>
     <dynamics damping="0.2"/>
-    <limit effort="100" velocity="1.0"/>
+    <limit effort="100" velocity="5.0"/>
   </joint>
   <!-- rear right wheel Link -->

Commit message: Setting velocity limit to 10 as it is defined in rad/s and we changed the turbo setting.

File: urdf/cmexa/cmexa_description.urdf.xacro (robot description, xacro)
@@ -64,5 +64,5 @@
     <axis xyz="0 1 0"/>
     <dynamics damping="0.2"/>
-    <limit effort="100" velocity="5.0"/>
+    <limit effort="100" velocity="10.0"/>
   </joint>
   <!-- Front right wheel -->
@@ -73,5 +73,5 @@
     <axis xyz="0 1 0"/>
     <dynamics damping="0.2"/>
-    <limit effort="100" velocity="5.0"/>
+    <limit effort="100" velocity="10.0"/>
   </joint>
   <!-- front right wheel Link -->
@@ -106,5 +106,5 @@
     <axis xyz="0 1 0"/>
     <dynamics damping="0.2"/>
-    <limit effort="100" velocity="5.0"/>
+    <limit effort="100" velocity="10.0"/>
   </joint>
   <!-- rear left wheel Link -->
@@ -139,5 +139,5 @@
     <axis xyz="0 1 0"/>
     <dynamics damping="0.2"/>
-    <limit effort="100" velocity="5.0"/>
+    <limit effort="100" velocity="10.0"/>
   </joint>
   <!-- rear right wheel Link -->

Commit message: Setting velocity limit to 20 as it is defined in rad/s and we changed the turbo setting.

File: urdf/cmexa/cmexa_description.urdf.xacro (robot description, xacro)
@@ -64,5 +64,5 @@
     <axis xyz="0 1 0"/>
     <dynamics damping="0.2"/>
-    <limit effort="100" velocity="10.0"/>
+    <limit effort="100" velocity="20.0"/>
   </joint>
   <!-- Front right wheel -->
@@ -73,5 +73,5 @@
     <axis xyz="0 1 0"/>
     <dynamics damping="0.2"/>
-    <limit effort="100" velocity="10.0"/>
+    <limit effort="100" velocity="20.0"/>
   </joint>
   <!-- front right wheel Link -->
@@ -106,5 +106,5 @@
     <axis xyz="0 1 0"/>
     <dynamics damping="0.2"/>
-    <limit effort="100" velocity="10.0"/>
+    <limit effort="100" velocity="20.0"/>
   </joint>
   <!-- rear left wheel Link -->
@@ -139,5 +139,5 @@
     <axis xyz="0 1 0"/>
     <dynamics damping="0.2"/>
-    <limit effort="100" velocity="10.0"/>
+    <limit effort="100" velocity="20.0"/>
   </joint>
   <!-- rear right wheel Link -->

Commit message: Setting velocity limit to 25 as it is defined in rad/s and we changed the turbo setting.

File: urdf/cmexa/cmexa_description.urdf.xacro (robot description, xacro)
@@ -64,5 +64,5 @@
     <axis xyz="0 1 0"/>
     <dynamics damping="0.2"/>
-    <limit effort="100" velocity="20.0"/>
+    <limit effort="100" velocity="25.0"/>
   </joint>
   <!-- Front right wheel -->
@@ -73,5 +73,5 @@
     <axis xyz="0 1 0"/>
     <dynamics damping="0.2"/>
-    <limit effort="100" velocity="20.0"/>
+    <limit effort="100" velocity="25.0"/>
   </joint>
   <!-- front right wheel Link -->
@@ -106,5 +106,5 @@
     <axis xyz="0 1 0"/>
     <dynamics damping="0.2"/>
-    <limit effort="100" velocity="20.0"/>
+    <limit effort="100" velocity="25.0"/>
   </joint>
   <!-- rear left wheel Link -->
@@ -139,5 +139,5 @@
     <axis xyz="0 1 0"/>
     <dynamics damping="0.2"/>
-    <limit effort="100" velocity="20.0"/>
+    <limit effort="100" velocity="25.0"/>
   </joint>
   <!-- rear right wheel Link -->

Commit message: Adding transmission for gear ratio 5:1

File: urdf/cmexa/cmexa_description.urdf.xacro (robot description, xacro)
@@ -66,4 +66,15 @@
     <limit effort="100" velocity="25.0"/>
   </joint>
+  <!-- Transmission for FRONT LEFT WHEEL -->
+  <transmission name="${prefix}front_left_wheel_trans">
+   <type>transmission_interface/SimpleTransmission</type>
+   <joint name="${prefix}front_left_wheel_joint">
+     <hardwareInterface>hardware_interface/VelocityJointInterface</hardwareInterface>
+   </joint>
+   <actuator name="${prefix}front_left_motor">
+     <hardwareInterface>hardware_interface/VelocityJointInterface</hardwareInterface>
+     <mechanicalReduction>${gear_ratio}</mechanicalReduction>
+   </actuator>
+</transmission>
   <!-- Front right wheel -->
   <joint name="${prefix}front_right_wheel_joint" type="continuous">
@@ -75,4 +86,15 @@
     <limit effort="100" velocity="25.0"/>
   </joint>
+  <!-- Transmission for FRONT RIGHT WHEEL -->
+  <transmission name="${prefix}front_right_wheel_trans">
+   <type>transmission_interface/SimpleTransmission</type>
+   <joint name="${prefix}front_right_wheel_joint">
+     <hardwareInterface>hardware_interface/VelocityJointInterface</hardwareInterface>
+   </joint>
+   <actuator name="${prefix}front_right_motor">
+     <hardwareInterface>hardware_interface/VelocityJointInterface</hardwareInterface>
+     <mechanicalReduction>${gear_ratio}</mechanicalReduction>
+   </actuator>
+  </transmission>
   <!-- front right wheel Link -->
   <link name="${prefix}front_right_wheel">
@@ -108,4 +130,15 @@
     <limit effort="100" velocity="25.0"/>
   </joint>
+   <!-- Transmission for REAR LEFT WHEEL -->
+   <transmission name="${prefix}rear_left_wheel_trans">
+     <type>transmission_interface/SimpleTransmission</type>
+     <joint name="${prefix}rear_left_wheel_joint">
+       <hardwareInterface>hardware_interface/VelocityJointInterface</hardwareInterface>
+     </joint>
+     <actuator name="${prefix}rear_left_motor">
+       <hardwareInterface>hardware_interface/VelocityJointInterface</hardwareInterface>
+       <mechanicalReduction>${gear_ratio}</mechanicalReduction>
+     </actuator>
+   </transmission>
   <!-- rear left wheel Link -->
   <link name="${prefix}rear_left_wheel">
@@ -141,4 +174,15 @@
     <limit effort="100" velocity="25.0"/>
   </joint>
+   <!-- Transmission for REAR RIGHT WHEEL -->
+   <transmission name="${prefix}rear_right_wheel_trans">
+     <type>transmission_interface/SimpleTransmission</type>
+     <joint name="${prefix}rear_right_wheel_joint">
+       <hardwareInterface>hardware_interface/VelocityJointInterface</hardwareInterface>
+     </joint>
+     <actuator name="${prefix}rear_right_motor">
+       <hardwareInterface>hardware_interface/VelocityJointInterface</hardwareInterface>
+       <mechanicalReduction>${gear_ratio}</mechanicalReduction>
+     </actuator>
+   </transmission>
   <!-- rear right wheel Link -->
   <link name="${prefix}rear_right_wheel">

File: urdf/cmexa/cmexa_properties.urdf.xacro (robot description, xacro)
@@ -11,6 +11,7 @@
   <xacro:property name="wheel_vertical_offset" value="0.01" />
   <xacro:property name="footprint_vertical_offset" value="0.025" />
-  <xacro:property name="wheel_radius" value="0.001" />
-  <xacro:property name="wheel_width" value="0.001" />
+  <xacro:property name="wheel_radius" value="0.05" />
+  <xacro:property name="wheel_width" value="0.05" />
+  <xacro:property name="gear_ratio" value="5.0"/>
   <xacro:property name="chassis_length" value="0.500" />
   <xacro:property name="chassis_width" value="0.350" />

Commit message: Lower limit to 15

File: urdf/cmexa/cmexa_description.urdf.xacro (robot description, xacro)
@@ -64,5 +64,5 @@
     <axis xyz="0 1 0"/>
     <dynamics damping="0.2"/>
-    <limit effort="100" velocity="25.0"/>
+    <limit effort="100" velocity="15.0"/>
   </joint>
   <!-- Transmission for FRONT LEFT WHEEL -->
@@ -84,5 +84,5 @@
     <axis xyz="0 1 0"/>
     <dynamics damping="0.2"/>
-    <limit effort="100" velocity="25.0"/>
+    <limit effort="100" velocity="15.0"/>
   </joint>
   <!-- Transmission for FRONT RIGHT WHEEL -->
@@ -128,5 +128,5 @@
     <axis xyz="0 1 0"/>
     <dynamics damping="0.2"/>
-    <limit effort="100" velocity="25.0"/>
+    <limit effort="100" velocity="15.0"/>
   </joint>
    <!-- Transmission for REAR LEFT WHEEL -->
@@ -172,5 +172,5 @@
     <axis xyz="0 1 0"/>
     <dynamics damping="0.2"/>
-    <limit effort="100" velocity="25.0"/>
+    <limit effort="100" velocity="15.0"/>
   </joint>
    <!-- Transmission for REAR RIGHT WHEEL -->
