Commit message: Corrected cmexa urdf xacro macros building the correct urdf links.

File: urdf/cmexa/cmexa.urdf.xacro (robot description, xacro)
@@ -4,11 +4,21 @@
     <xacro:arg name="prefix" default="" />
     <xacro:arg name="use_mock_hardware" default="false" />
-    <xacro:include filename="$(find cmeresearch_description)/urdf/cmexa/cmexa_description.urdf.xacro" />
+    <!-- Robot constants and properties -->
+    <xacro:include filename="$(find cmeresearch_description)/urdf/cmexa/cmexa_properties.urdf.xacro" />
     <!-- Import Rviz colors -->
     <xacro:include filename="$(find cmeresearch_description)/urdf/materials.xacro" />
+    <!-- Import robot description -->
+    <xacro:include filename="$(find cmeresearch_description)/urdf/cmexa/cmexa_description.urdf.xacro" />
     <!-- Import ros2_control description -->
     <xacro:include filename="$(find cmeresearch_description)/urdf/cmexa/cmexa_mecanum.ros2_control.xacro" />
-    <xacro:cmexa prefix="$(arg prefix)" />
-    <xacro:cmexa_ros2_control
-            name="CMEXA" prefix="$(arg prefix)" use_mock_hardware="$(arg use_mock_hardware)"/>
+    <!-- Instantiate the robot -->
+    <xacro:macro name="cmexa_robot" params="prefix">
+        <!-- Create the robot chassis and wheels -->
+        <xacro:cmexa prefix="${prefix}" />
+        <!-- Add ros2_control -->
+        <xacro:cmexa_ros2_control
+                name="CMEXA" prefix="${prefix}" use_mock_hardware="$(arg use_mock_hardware)"/>
+    </xacro:macro>
+    <!-- Create the robot instance -->
+    <xacro:cmexa_robot prefix="$(arg prefix)" />
 </robot>

File: urdf/cmexa/cmexa_description.urdf.xacro (robot description, xacro)
@@ -1,7 +1,5 @@
 <?xml version="1.0"?>
 <robot xmlns:xacro="http://www.ros.org/wiki/xacro">
-  <xacro:macro name="cmexa" params="prefix">
-  <!-- Robot constants and properties -->
-  <xacro:include filename="$(find cmeresearch_description)/urdf/cmexa/cmexa_properties.urdf.xacro" />
+ <xacro:macro name="cmexa" params="prefix">
   <xacro:property name="z_offset" value="-${chassis_height/2}" /> <!-- Space btw top of beam and the each joint -->
   <xacro:property name="wheel_mass" value="0.3"/>
@@ -170,4 +168,4 @@
       </inertial>
     </link>
-  </xacro:macro>
+ </xacro:macro>
 </robot>

Commit message: Corrected cmexa urdf (wrong position in chassis leads to complex errors in launch and yaml file.)

File: urdf/cmexa/cmexa.urdf.xacro (robot description, xacro)
@@ -2,23 +2,19 @@
 <!-- Basic mecanum drive mobile base -->
 <robot xmlns:xacro="http://www.ros.org/wiki/xacro" name="mecanumdrive_robot">
-    <xacro:arg name="prefix" default="" />
-    <xacro:arg name="use_mock_hardware" default="false" />
-    <!-- Robot constants and properties -->
-    <xacro:include filename="$(find cmeresearch_description)/urdf/cmexa/cmexa_properties.urdf.xacro" />
-    <!-- Import Rviz colors -->
-    <xacro:include filename="$(find cmeresearch_description)/urdf/materials.xacro" />
-    <!-- Import robot description -->
-    <xacro:include filename="$(find cmeresearch_description)/urdf/cmexa/cmexa_description.urdf.xacro" />
-    <!-- Import ros2_control description -->
-    <xacro:include filename="$(find cmeresearch_description)/urdf/cmexa/cmexa_mecanum.ros2_control.xacro" />
-    <!-- Instantiate the robot -->
-    <xacro:macro name="cmexa_robot" params="prefix">
-        <!-- Create the robot chassis and wheels -->
-        <xacro:cmexa prefix="${prefix}" />
-        <!-- Add ros2_control -->
-        <xacro:cmexa_ros2_control
-                name="CMEXA" prefix="${prefix}" use_mock_hardware="$(arg use_mock_hardware)"/>
-    </xacro:macro>
-    <!-- Create the robot instance -->
-    <xacro:cmexa_robot prefix="$(arg prefix)" />
+  <!-- Parameters -->
+  <xacro:arg name="prefix" default="" />
+  <xacro:arg name="use_mock_hardware" default="false" />
+  <!-- Import robot description -->
+  <xacro:include filename="$(find cmeresearch_description)/urdf/cmexa/cmexa_description.urdf.xacro" />
+  <!-- Robot constants and properties -->
+  <xacro:include filename="$(find cmeresearch_description)/urdf/cmexa/cmexa_properties.urdf.xacro" />
+  <!-- Import Rviz colors -->
+  <xacro:include filename="$(find cmeresearch_description)/urdf/materials.xacro" />
+  <!-- Import ros2_control description -->
+  <xacro:include filename="$(find cmeresearch_description)/urdf/cmexa/cmexa_mecanum.ros2_control.xacro" />
+  <!-- Instantiate the robot -->
+  <xacro:cmexa prefix="$(arg prefix)" />
+  <!-- Add ros2_control -->
+  <xacro:cmexa_ros2_control
+    name="Cmexa" prefix="$(arg prefix)" use_mock_hardware="$(arg use_mock_hardware)"/>
 </robot>

File: urdf/cmexa/cmexa_description.urdf.xacro (robot description, xacro)
@@ -2,9 +2,8 @@
 <robot xmlns:xacro="http://www.ros.org/wiki/xacro">
  <xacro:macro name="cmexa" params="prefix">
-  <xacro:property name="z_offset" value="-${chassis_height/2}" /> <!-- Space btw top of beam and the each joint -->
-  <xacro:property name="wheel_mass" value="0.3"/>
     <!-- Base Link -->
-  <link name="${prefix}base_link"></link>
-  <joint name="base_link_joint" type="fixed">
+  <link name="${prefix}base_link">
+  </link>
+  <joint name="${prefix}base_link_joint" type="fixed">
     <origin xyz="0 0 ${wheel_radius/2}" rpy="0 0 0" />
     <parent link="${prefix}base_link"/>
@@ -20,5 +19,5 @@
     </visual>
     <collision>
-      <origin xyz="${chassis_length/2} ${chassis_width/2} ${chassis_height/2}"/>
+      <origin xyz="${chassis_length/2} ${-chassis_width/2} 0"/>
       <geometry>
         <box size="${chassis_length} ${chassis_width} ${chassis_height}"/>
@@ -26,8 +25,6 @@
     </collision>
     <inertial>
-      <!-- Center of mass -->
       <origin xyz="0.012  0.002 0.067" rpy="0 0 0"/>
       <mass value="16.523"/>
-      <!-- Moments of inertia: ( chassis without wheels ) -->
       <inertia
         ixx="0.3136" ixy="-0.0008" ixz="0.0164"
@@ -37,135 +34,135 @@
   </link>
     <!-- Front left wheel -->
-    <joint name="${prefix}front_left_wheel_joint" type="continuous">
-      <parent link="${prefix}base_link"/>
-      <child link="${prefix}front_left_wheel"/>
-      <origin xyz="${wheelbase/2} ${track/2} ${wheel_radius/2}" rpy="0 0 0"/>
-      <axis xyz="0 1 0"/>
-      <dynamics damping="0.2"/>
-      <limit effort="100" velocity="1.0"/>
-    </joint>
-    <!-- front left wheel Link -->
-    <link name="${prefix}front_left_wheel">
-      <collision>
-        <origin xyz="0 0 0" rpy="${PI/2} 0 0"/>
-        <geometry>
-          <cylinder length="${wheel_width}" radius="${wheel_radius}"/>
-        </geometry>
-      </collision>
-      <visual>
-        <origin xyz="0 0 0" rpy="${PI/2} 0 0"/>
-        <geometry>
-          <cylinder length="${wheel_width}" radius="${wheel_radius}"/>
-        </geometry>
-        <material name="black"/>
-      </visual>
-      <inertial>
-        <origin xyz="0 0 0" rpy="${PI/2} 0 0"/>
-        <mass value="${wheel_mass}"/>
-        <inertia
-                ixx="${wheel_mass / 12.0 * (3*wheel_radius*wheel_radius + wheel_width*wheel_width)}" ixy="0.0" ixz="0.0"
-                iyy="${wheel_mass / 12.0 * (3*wheel_radius*wheel_radius + wheel_width*wheel_width)}" iyz="0.0"
-                izz="${wheel_mass / 2.0 * wheel_radius*wheel_radius}"/>
-      </inertial>
-    </link>
-    <!-- Front right wheel -->
-    <joint name="${prefix}front_right_wheel_joint" type="continuous">
-      <parent link="${prefix}base_link"/>
-      <child link="${prefix}front_right_wheel"/>
-      <origin xyz="${-wheelbase/2} ${track/2} ${wheel_radius/2}" rpy="0 0 0"/>
-      <axis xyz="0 1 0"/>
-      <dynamics damping="0.2"/>
-      <limit effort="100" velocity="1.0"/>
-    </joint>
-    <!-- front right wheel Link -->
-    <link name="${prefix}front_right_wheel">
-      <collision>
-        <origin xyz="0 0 0" rpy="${PI/2} 0 0"/>
-        <geometry>
-          <cylinder length="${wheel_width}" radius="${wheel_radius}"/>
-        </geometry>
-      </collision>
-      <visual>
-        <origin xyz="0 0 0" rpy="${PI/2} 0 0"/>
-        <geometry>
-          <cylinder length="${wheel_width}" radius="${wheel_radius}"/>
-        </geometry>
-        <material name="black"/>
-      </visual>
-      <inertial>
-        <origin xyz="0 0 0" rpy="${PI/2} 0 0"/>
-        <mass value="${wheel_mass}"/>
-        <inertia
-                ixx="${wheel_mass / 12.0 * (3*wheel_radius*wheel_radius + wheel_width*wheel_width)}" ixy="0.0" ixz="0.0"
-                iyy="${wheel_mass / 12.0 * (3*wheel_radius*wheel_radius + wheel_width*wheel_width)}" iyz="0.0"
-                izz="${wheel_mass / 2.0 * wheel_radius*wheel_radius}"/>
-      </inertial>
-    </link>
-    <!-- rear left wheel -->
-    <joint name="${prefix}rear_left_wheel_joint" type="continuous">
-      <parent link="${prefix}base_link"/>
-      <child link="${prefix}rear_left_wheel"/>
-      <origin xyz="${wheelbase/2} ${-track/2} ${wheel_radius/2}" rpy="0 0 0"/>
-      <axis xyz="0 1 0"/>
-      <dynamics damping="0.2"/>
-      <limit effort="100" velocity="1.0"/>
-    </joint>
-    <!-- rear left wheel Link -->
-    <link name="${prefix}rear_left_wheel">
-      <collision>
-        <origin xyz="0 0 0" rpy="${PI/2} 0 0"/>
-        <geometry>
-          <cylinder length="${wheel_width}" radius="${wheel_radius}"/>
-        </geometry>
-      </collision>
-      <visual>
-        <origin xyz="0 0 0" rpy="${PI/2} 0 0"/>
-        <geometry>
-          <cylinder length="${wheel_width}" radius="${wheel_radius}"/>
-        </geometry>
-        <material name="black"/>
-      </visual>
-      <inertial>
-        <origin xyz="0 0 0" rpy="${PI/2} 0 0"/>
-        <mass value="${wheel_mass}"/>
-        <inertia
-                ixx="${wheel_mass / 12.0 * (3*wheel_radius*wheel_radius + wheel_width*wheel_width)}" ixy="0.0" ixz="0.0"
-                iyy="${wheel_mass / 12.0 * (3*wheel_radius*wheel_radius + wheel_width*wheel_width)}" iyz="0.0"
-                izz="${wheel_mass / 2.0 * wheel_radius*wheel_radius}"/>
-      </inertial>
-    </link>
-    <!-- rear right wheel -->
-    <joint name="${prefix}rear_right_wheel_joint" type="continuous">
-      <parent link="${prefix}base_link"/>
-      <child link="${prefix}rear_right_wheel"/>
-      <origin xyz="${-wheelbase/2} ${-track/2} ${wheel_radius/2}" rpy="0 0 0"/>
-      <axis xyz="0 1 0"/>
-      <dynamics damping="0.2"/>
-      <limit effort="100" velocity="1.0"/>
-    </joint>
-    <!-- rear right wheel Link -->
-    <link name="${prefix}rear_right_wheel">
-      <collision>
-        <origin xyz="0 0 0" rpy="${PI/2} 0 0"/>
-        <geometry>
-          <cylinder length="${wheel_width}" radius="${wheel_radius}"/>
-        </geometry>
-      </collision>
-      <visual>
-        <origin xyz="0 0 0" rpy="${PI/2} 0 0"/>
-        <geometry>
-          <cylinder length="${wheel_width}" radius="${wheel_radius}"/>
-        </geometry>
-        <material name="black"/>
-      </visual>
-      <inertial>
-        <origin xyz="0 0 0" rpy="${PI/2} 0 0"/>
-        <mass value="${wheel_mass}"/>
-        <inertia
-                ixx="${wheel_mass / 12.0 * (3*wheel_radius*wheel_radius + wheel_width*wheel_width)}" ixy="0.0" ixz="0.0"
-                iyy="${wheel_mass / 12.0 * (3*wheel_radius*wheel_radius + wheel_width*wheel_width)}" iyz="0.0"
-                izz="${wheel_mass / 2.0 * wheel_radius*wheel_radius}"/>
-      </inertial>
-    </link>
+  <joint name="${prefix}front_left_wheel_joint" type="continuous">
+    <parent link="${prefix}base_link"/>
+    <child link="${prefix}front_left_wheel"/>
+    <origin xyz="${wheelbase/2} ${track/2} ${wheel_radius/2}" rpy="0 0 0"/>
+    <axis xyz="0 1 0"/>
+    <dynamics damping="0.2"/>
+    <limit effort="100" velocity="1.0"/>
+  </joint>
+  <!-- front left wheel Link -->
+  <link name="${prefix}front_left_wheel">
+    <collision>
+      <origin xyz="0 0 0" rpy="${PI/2} 0 0"/>
+      <geometry>
+        <cylinder length="${wheel_width}" radius="${wheel_radius}"/>
+      </geometry>
+    </collision>
+    <visual>
+      <origin xyz="0 0 0" rpy="${PI/2} 0 0"/>
+      <geometry>
+        <cylinder length="${wheel_width}" radius="${wheel_radius}"/>
+      </geometry>
+      <material name="black"/>
+    </visual>
+    <inertial>
+      <origin xyz="0 0 0" rpy="${PI/2} 0 0"/>
+      <mass value="${wheel_mass}"/>
+      <inertia
+              ixx="${wheel_mass / 12.0 * (3*wheel_radius*wheel_radius + wheel_width*wheel_width)}" ixy="0.0" ixz="0.0"
+              iyy="${wheel_mass / 12.0 * (3*wheel_radius*wheel_radius + wheel_width*wheel_width)}" iyz="0.0"
+              izz="${wheel_mass / 2.0 * wheel_radius*wheel_radius}"/>
+    </inertial>
+  </link>
+  <!-- Front right wheel -->
+  <joint name="${prefix}front_right_wheel_joint" type="continuous">
+    <parent link="${prefix}base_link"/>
+    <child link="${prefix}front_right_wheel"/>
+    <origin xyz="${-wheelbase/2} ${track/2} ${wheel_radius/2}" rpy="0 0 0"/>
+    <axis xyz="0 1 0"/>
+    <dynamics damping="0.2"/>
+    <limit effort="100" velocity="1.0"/>
+  </joint>
+  <!-- front right wheel Link -->
+  <link name="${prefix}front_right_wheel">
+    <collision>
+      <origin xyz="0 0 0" rpy="${PI/2} 0 0"/>
+      <geometry>
+        <cylinder length="${wheel_width}" radius="${wheel_radius}"/>
+      </geometry>
+    </collision>
+    <visual>
+      <origin xyz="0 0 0" rpy="${PI/2} 0 0"/>
+      <geometry>
+        <cylinder length="${wheel_width}" radius="${wheel_radius}"/>
+      </geometry>
+      <material name="black"/>
+    </visual>
+    <inertial>
+      <origin xyz="0 0 0" rpy="${PI/2} 0 0"/>
+      <mass value="${wheel_mass}"/>
+      <inertia
+              ixx="${wheel_mass / 12.0 * (3*wheel_radius*wheel_radius + wheel_width*wheel_width)}" ixy="0.0" ixz="0.0"
+              iyy="${wheel_mass / 12.0 * (3*wheel_radius*wheel_radius + wheel_width*wheel_width)}" iyz="0.0"
+              izz="${wheel_mass / 2.0 * wheel_radius*wheel_radius}"/>
+    </inertial>
+  </link>
+  <!-- rear left wheel -->
+  <joint name="${prefix}rear_left_wheel_joint" type="continuous">
+    <parent link="${prefix}base_link"/>
+    <child link="${prefix}rear_left_wheel"/>
+    <origin xyz="${wheelbase/2} ${-track/2} ${wheel_radius/2}" rpy="0 0 0"/>
+    <axis xyz="0 1 0"/>
+    <dynamics damping="0.2"/>
+    <limit effort="100" velocity="1.0"/>
+  </joint>
+  <!-- rear left wheel Link -->
+  <link name="${prefix}rear_left_wheel">
+    <collision>
+      <origin xyz="0 0 0" rpy="${PI/2} 0 0"/>
+      <geometry>
+        <cylinder length="${wheel_width}" radius="${wheel_radius}"/>
+      </geometry>
+    </collision>
+    <visual>
+      <origin xyz="0 0 0" rpy="${PI/2} 0 0"/>
+      <geometry>
+        <cylinder length="${wheel_width}" radius="${wheel_radius}"/>
+      </geometry>
+      <material name="black"/>
+    </visual>
+    <inertial>
+      <origin xyz="0 0 0" rpy="${PI/2} 0 0"/>
+      <mass value="${wheel_mass}"/>
+      <inertia
+              ixx="${wheel_mass / 12.0 * (3*wheel_radius*wheel_radius + wheel_width*wheel_width)}" ixy="0.0" ixz="0.0"
+              iyy="${wheel_mass / 12.0 * (3*wheel_radius*wheel_radius + wheel_width*wheel_width)}" iyz="0.0"
+              izz="${wheel_mass / 2.0 * wheel_radius*wheel_radius}"/>
+    </inertial>
+  </link>
+  <!-- rear right wheel -->
+  <joint name="${prefix}rear_right_wheel_joint" type="continuous">
+    <parent link="${prefix}base_link"/>
+    <child link="${prefix}rear_right_wheel"/>
+    <origin xyz="${-wheelbase/2} ${-track/2} ${wheel_radius/2}" rpy="0 0 0"/>
+    <axis xyz="0 1 0"/>
+    <dynamics damping="0.2"/>
+    <limit effort="100" velocity="1.0"/>
+  </joint>
+  <!-- rear right wheel Link -->
+  <link name="${prefix}rear_right_wheel">
+    <collision>
+      <origin xyz="0 0 0" rpy="${PI/2} 0 0"/>
+      <geometry>
+        <cylinder length="${wheel_width}" radius="${wheel_radius}"/>
+      </geometry>
+    </collision>
+    <visual>
+      <origin xyz="0 0 0" rpy="${PI/2} 0 0"/>
+      <geometry>
+        <cylinder length="${wheel_width}" radius="${wheel_radius}"/>
+      </geometry>
+      <material name="black"/>
+    </visual>
+    <inertial>
+      <origin xyz="0 0 0" rpy="${PI/2} 0 0"/>
+      <mass value="${wheel_mass}"/>
+      <inertia
+              ixx="${wheel_mass / 12.0 * (3*wheel_radius*wheel_radius + wheel_width*wheel_width)}" ixy="0.0" ixz="0.0"
+              iyy="${wheel_mass / 12.0 * (3*wheel_radius*wheel_radius + wheel_width*wheel_width)}" iyz="0.0"
+              izz="${wheel_mass / 2.0 * wheel_radius*wheel_radius}"/>
+    </inertial>
+  </link>
  </xacro:macro>
 </robot>

File: urdf/cmexa/cmexa_mecanum.ros2_control.xacro (robot description, xacro)
@@ -1,40 +1,40 @@
 <?xml version="1.0"?>
 <robot xmlns:xacro="http://www.ros.org/wiki/xacro">
-    <xacro:macro name="cmexa_ros2_control" params="name prefix use_mock_hardware">
-        <ros2_control name="${name}" type="system">
-            <xacro:unless value="${use_mock_hardware}">
-                <hardware>
-                    <plugin>cmexa_base/CmexaMecanumBotSystemHardware</plugin>
-                    <param name="example_param_hw_start_duration_sec">0</param>
-                    <param name="example_param_hw_stop_duration_sec">3.0</param>
-                </hardware>
-            </xacro:unless>
-            <xacro:if value="${use_mock_hardware}">
-                <hardware>
-                    <plugin>mock_components/GenericSystem</plugin>
-                    <param name="calculate_dynamics">true</param>
-                </hardware>
-            </xacro:if>
-            <joint name="${prefix}front_left_wheel_joint">
-                <command_interface name="velocity"/>
-                <state_interface name="position"/>
-                <state_interface name="velocity"/>
-            </joint>
-            <joint name="${prefix}rear_left_wheel_joint">
-                <command_interface name="velocity"/>
-                <state_interface name="position"/>
-                <state_interface name="velocity"/>
-            </joint>
-            <joint name="${prefix}front_right_wheel_joint">
-                <command_interface name="velocity"/>
-                <state_interface name="position"/>
-                <state_interface name="velocity"/>
-            </joint>
-            <joint name="${prefix}rear_right_wheel_joint">
-                <command_interface name="velocity"/>
-                <state_interface name="position"/>
-                <state_interface name="velocity"/>
-            </joint>
-        </ros2_control>
-    </xacro:macro>
+  <xacro:macro name="cmexa_ros2_control" params="name prefix use_mock_hardware">
+    <ros2_control name="${name}" type="system">
+      <xacro:unless value="${use_mock_hardware}">
+        <hardware>
+          <plugin>cmexa_base/CmexaMecanumBotSystemHardware</plugin>
+            <param name="example_param_hw_start_duration_sec">0</param>
+            <param name="example_param_hw_stop_duration_sec">3.0</param>
+        </hardware>
+        </xacro:unless>
+        <xacro:if value="${use_mock_hardware}">
+          <hardware>
+            <plugin>mock_components/GenericSystem</plugin>
+            <param name="calculate_dynamics">true</param>
+          </hardware>
+        </xacro:if>
+        <joint name="${prefix}front_left_wheel_joint">
+          <command_interface name="velocity"/>
+          <state_interface name="position"/>
+          <state_interface name="velocity"/>
+        </joint>
+        <joint name="${prefix}rear_left_wheel_joint">
+          <command_interface name="velocity"/>
+          <state_interface name="position"/>
+          <state_interface name="velocity"/>
+        </joint>
+        <joint name="${prefix}front_right_wheel_joint">
+          <command_interface name="velocity"/>
+          <state_interface name="position"/>
+          <state_interface name="velocity"/>
+        </joint>
+        <joint name="${prefix}rear_right_wheel_joint">
+          <command_interface name="velocity"/>
+          <state_interface name="position"/>
+          <state_interface name="velocity"/>
+        </joint>
+      </ros2_control>
+  </xacro:macro>
 </robot>

File: urdf/cmexa/cmexa_properties.urdf.xacro (robot description, xacro)
@@ -16,6 +16,8 @@
   <xacro:property name="chassis_width" value="0.350" />
   <xacro:property name="chassis_height" value="0.300" />
-  <xacro:property name="chassis_mass" value="0.3" /> <!-- correct this later -->
+  <xacro:property name="chassis_mass" value="0.3" />
   <xacro:property name="dummy_inertia" value="1e-09"/>
   <xacro:property name="mount_spacing" value="0.120" />
+  <xacro:property name="z_offset" value="-${chassis_height/2}" /> <!-- Space btw top of beam and the each joint -->
+  <xacro:property name="wheel_mass" value="0.3"/>
 </robot>

File: urdf/cmexaiii/cmexaiii.urdf.xacro (robot description, xacro)
@@ -4,11 +4,21 @@
     <xacro:arg name="prefix" default="" />
     <xacro:arg name="use_mock_hardware" default="false" />
-    <xacro:include filename="$(find cmeresearch_description)/urdf/cmexaiii/cmexaiii_description.urdf.xacro" />
+    <!-- Robot constants and properties -->
+    <xacro:include filename="$(find cmeresearch_description)/urdf/cmexaiii/cmexaiii_properties.urdf.xacro" />
     <!-- Import Rviz colors -->
     <xacro:include filename="$(find cmeresearch_description)/urdf/materials.xacro" />
+    <!-- Import robot description -->
+    <xacro:include filename="$(find cmeresearch_description)/urdf/cmexaiii/cmexaiii_description.urdf.xacro" />
     <!-- Import ros2_control description -->
     <xacro:include filename="$(find cmeresearch_description)/urdf/cmexaiii/cmexaiii_mecanum.ros2_control.xacro" />
-    <xacro:cmexaiii prefix="$(arg prefix)" />
-    <xacro:cmexaiii_ros2_control
-            name="CMEXAIII" prefix="$(arg prefix)" use_mock_hardware="$(arg use_mock_hardware)"/>
+    <!-- Instantiate the robot -->
+    <xacro:macro name="cmexaiii_robot" params="prefix">
+        <!-- Create the robot chassis and wheels -->
+        <xacro:cmexa prefix="${prefix}" />
+        <!-- Add ros2_control -->
+        <xacro:cmexa_ros2_control
+                name="CMEXAIII" prefix="${prefix}" use_mock_hardware="$(arg use_mock_hardware)"/>
+    </xacro:macro>
+    <!-- Create the robot instance -->
+    <xacro:cmexaiii_robot prefix="$(arg prefix)" />
 </robot>

File: urdf/cmexaiii/cmexaiii_description.urdf.xacro (robot description, xacro)
@@ -2,6 +2,4 @@
 <robot xmlns:xacro="http://www.ros.org/wiki/xacro">
   <xacro:macro name="cmexaiii" params="prefix">
-  <!-- Robot constants and properties -->
-  <xacro:include filename="$(find cmeresearch_description)/urdf/cmexaiii/cmexaiii_properties.urdf.xacro" />
   <xacro:property name="z_offset" value="-${chassis_height/2}" /> <!-- Space btw top of beam and the each joint -->
   <xacro:property name="wheel_mass" value="0.3"/>

File: urdf/materials.xacro (robot description, xacro)
@@ -7,3 +7,4 @@
   <material name="green"><color rgba="0.25 0.75 0.25 1.0" /></material>
   <material name="orange"><color rgba="0.92 0.33 0.02 1.0" /></material>
+  <material name="white"><color rgba="1.0 1.0 1.0 1.0"/></material>
 </robot>
