Commit message: Added gear ratio and steps per revolution as properties and updated mecanum control configurations in URDF Xacros.

File: urdf/cmexa/cmexa_mecanum.ros2_control.xacro (robot description, xacro)
@@ -8,5 +8,9 @@
             <param name="example_param_hw_start_duration_sec">0</param>
             <param name="example_param_hw_stop_duration_sec">3.0</param>
-            <param name="gear_ratio">5.0</param>
+            <param name="gear_ratio">${gear_ratio}</param>
+            <param name="wheel_radius">${wheel_radius}</param>
+            <param name="wheel_separation_x">${wheelbase}</param>
+            <param name="wheel_separation_y">${track}</param>
+            <param name="steps_per_revolution">200.0</param>
         </hardware>
         </xacro:unless>

File: urdf/cmexaiii/cmexaiii_mecanum.ros2_control.xacro (robot description, xacro)
@@ -8,5 +8,9 @@
                     <param name="example_param_hw_start_duration_sec">0</param>
                     <param name="example_param_hw_stop_duration_sec">3.0</param>
-                    <param name="gear_ratio">5.0</param>
+                    <param name="gear_ratio">${gear_ratio}</param>
+                    <param name="wheel_radius">${wheel_radius}</param>
+                    <param name="wheel_separation_x">${wheelbase}</param>
+                    <param name="wheel_separation_y">${track}</param>
+                    <param name="steps_per_revolution">${steps_per_revolution}</param>
                 </hardware>
             </xacro:unless>

File: urdf/cmexaiii/cmexaiii_properties.urdf.xacro (robot description, xacro)
@@ -8,4 +8,6 @@
        example: distance between wheel_front_right and wheel_front_left -->
   <xacro:property name="track" value="0.354" />
+  <xacro:property name="gear_ratio" value="5.0" />
+  <xacro:property name="steps_per_revolution" value="200.0" />
   <!-- vertical offset means height -->
   <xacro:property name="wheel_vertical_offset" value="0.01" />
