Commit message: feat(urdf): pass step_resolution to ros2_control hardware_parameter
The cmexa_base hardware interface needs step_resolution alongside
steps_per_revolution and gear_ratio to correctly convert bricklet
microsteps/s feedback back into wheel rad/s for odometry. Without it
the reported wheel velocity is off by a factor of step_resolution
(currently 8x too high), which silently corrupts /odom and
slam_toolbox map scale.

Adds a step_resolution xacro property (8 = 1/8 microstep, matching the
bricklet config in cmeresearch_stepper_driver) to both cmexaiii and
cmexa robot_properties files, and a matching <param> entry in their
ros2_control xacros. cmexa also gets a steps_per_revolution property
so both vars are defined symbolically instead of hardcoded.

File: urdf/cmexa/robot_mecanum.ros2_control.xacro (robot description, xacro)
@@ -12,5 +12,6 @@
             <param name="wheel_separation_x">${wheelbase}</param>
             <param name="wheel_separation_y">${track}</param>
-            <param name="steps_per_revolution">200.0</param>
+            <param name="steps_per_revolution">${steps_per_revolution}</param>
+            <param name="step_resolution">${step_resolution}</param>
         </hardware>
         </xacro:unless>

File: urdf/cmexa/robot_properties.urdf.xacro (robot description, xacro)
@@ -14,4 +14,8 @@
   <xacro:property name="wheel_width" value="0.05" />
   <xacro:property name="gear_ratio" value="5.0"/>
+  <xacro:property name="steps_per_revolution" value="200.0"/>
+  <!-- Bricklet microstep mode: must match SILENT_STEPPER_V2_STEP_RESOLUTION_*
+       configured in cmeresearch_stepper_driver. 8 = 1/8 step (8 microsteps per full step). -->
+  <xacro:property name="step_resolution" value="8"/>
   <xacro:property name="chassis_length" value="0.500" />
   <xacro:property name="chassis_width" value="0.350" />

File: urdf/cmexaiii/robot_mecanum.ros2_control.xacro (robot description, xacro)
@@ -13,4 +13,5 @@
                     <param name="wheel_separation_y">${track}</param>
                     <param name="steps_per_revolution">${steps_per_revolution}</param>
+                    <param name="step_resolution">${step_resolution}</param>
                 </hardware>
             </xacro:unless>

File: urdf/cmexaiii/robot_properties.urdf.xacro (robot description, xacro)
@@ -10,4 +10,7 @@
   <xacro:property name="gear_ratio" value="5.0" />
   <xacro:property name="steps_per_revolution" value="200.0" />
+  <!-- Bricklet microstep mode: must match SILENT_STEPPER_V2_STEP_RESOLUTION_*
+       configured in cmeresearch_stepper_driver. 8 = 1/8 step (8 microsteps per full step). -->
+  <xacro:property name="step_resolution" value="8" />
   <!-- vertical offset means height -->
   <xacro:property name="wheel_vertical_offset" value="0.01" />
