Commit message: Adding CMEXB configs

File: urdf/cmexb/cmexb_diff.ros2_control.xacro (robot description, xacro)
@@ -5,5 +5,5 @@
       <xacro:unless value="${use_mock_hardware}">
         <hardware>
-          <plugin>cmexb_base/CmexbDiffBotSystemHardware</plugin>
+          <plugin>cmexa_base/CmexaDiffBotSystemHardware</plugin>
             <param name="example_param_hw_start_duration_sec">0</param>
             <param name="example_param_hw_stop_duration_sec">3.0</param>
@@ -17,9 +17,4 @@
           </hardware>
         </xacro:if>
-        <joint name="${prefix}front_left_wheel_joint">
-          <command_interface name="velocity"/>
-          <state_interface name="position"/>
-          <state_interface name="velocity"/>
-        </joint>
         <joint name="${prefix}rear_left_wheel_joint">
           <command_interface name="velocity"/>
@@ -32,9 +27,4 @@
           <state_interface name="velocity"/>
         </joint>
-        <joint name="${prefix}rear_right_wheel_joint">
-          <command_interface name="velocity"/>
-          <state_interface name="position"/>
-          <state_interface name="velocity"/>
-        </joint>
       </ros2_control>
   </xacro:macro>

Commit message: test

File: urdf/cmexb/cmexb_diff.ros2_control.xacro (robot description, xacro)
@@ -5,5 +5,5 @@
       <xacro:unless value="${use_mock_hardware}">
         <hardware>
-          <plugin>cmexa_base/CmexaDiffBotSystemHardware</plugin>
+          <plugin>cmexa_base/CmexBotSystemHardware</plugin>
             <param name="example_param_hw_start_duration_sec">0</param>
             <param name="example_param_hw_stop_duration_sec">3.0</param>
@@ -17,4 +17,9 @@
           </hardware>
         </xacro:if>
+        <joint name="${prefix}front_left_wheel_joint">
+          <command_interface name="velocity"/>
+          <state_interface name="position"/>
+          <state_interface name="velocity"/>
+        </joint>
         <joint name="${prefix}rear_left_wheel_joint">
           <command_interface name="velocity"/>
@@ -27,4 +32,9 @@
           <state_interface name="velocity"/>
         </joint>
+        <joint name="${prefix}rear_right_wheel_joint">
+          <command_interface name="velocity"/>
+          <state_interface name="position"/>
+          <state_interface name="velocity"/>
+        </joint>
       </ros2_control>
   </xacro:macro>
