Commit message: test

File: urdf/cmexb/cmexb_description.urdf.xacro (robot description, xacro)
@@ -81,5 +81,5 @@
     <parent link="${prefix}base_link"/>
     <child link="${prefix}front_right_wheel"/>
-    <origin xyz="${-wheelbase/2} ${track/2} ${wheel_radius/2}" rpy="0 0 0"/>
+    <origin xyz="${wheelbase/2} ${-track/2} ${wheel_radius/2}" rpy="0 0 0"/>
     <axis xyz="0 1 0"/>
     <dynamics damping="0.2"/>
@@ -125,5 +125,5 @@
     <parent link="${prefix}base_link"/>
     <child link="${prefix}rear_left_wheel"/>
-    <origin xyz="${wheelbase/2} ${-track/2} ${wheel_radius/2}" rpy="0 0 0"/>
+    <origin xyz="${-wheelbase/2} ${track/2} ${wheel_radius/2}" rpy="0 0 0"/>
     <axis xyz="0 1 0"/>
     <dynamics damping="0.2"/>
