Commit message: test

File: urdf/cmexamini/cmexamini.urdf.xacro (robot description, xacro)
@@ -6,15 +6,15 @@
   <xacro:arg name="use_mock_hardware" default="false" />
   <!-- Import robot description -->
-  <xacro:include filename="$(find cmeresearch_description)/urdf/cmexb/cmexb_description.urdf.xacro" />
+  <xacro:include filename="$(find cmeresearch_description)/urdf/cmexamini/cmexamini_description.urdf.xacro" />
   <!-- Robot constants and properties -->
-  <xacro:include filename="$(find cmeresearch_description)/urdf/cmexb/cmexb_properties.urdf.xacro" />
+  <xacro:include filename="$(find cmeresearch_description)/urdf/cmexamini/cmexamini_properties.urdf.xacro" />
   <!-- Import Rviz colors -->
   <xacro:include filename="$(find cmeresearch_description)/urdf/materials.xacro" />
   <!-- Import ros2_control description -->
-  <xacro:include filename="$(find cmeresearch_description)/urdf/cmexb/cmexb_diff.ros2_control.xacro" />
+  <xacro:include filename="$(find cmeresearch_description)/urdf/cmexamini/cmexamini_diff.ros2_control.xacro" />
   <!-- Instantiate the robot -->
   <xacro:cmexb prefix="$(arg prefix)" />
   <!-- Add ros2_control -->
-  <xacro:cmexb_ros2_control
-    name="Cmexb" prefix="$(arg prefix)" use_mock_hardware="$(arg use_mock_hardware)"/>
+  <xacro:cmexamini_ros2_control
+    name="CMEXAMINI" prefix="$(arg prefix)" use_mock_hardware="$(arg use_mock_hardware)"/>
 </robot>

File: urdf/cmexamini/cmexamini_description.urdf.xacro (robot description, xacro)
@@ -14,5 +14,5 @@
       <origin xyz="${chassis_length/2} ${-chassis_width/2} 0" rpy="0 0 ${PI/2}" />
       <geometry>
-        <mesh filename="package://cmeresearch_description/meshes/cmexb/cmexb-base.stl" scale="0.001 0.001 0.001"/>
+        <mesh filename="package://cmeresearch_description/meshes/cmexamini/cmexamini-base.stl" scale="0.001 0.001 0.001"/>
       </geometry>
       <material name="dark_grey" />
@@ -36,5 +36,5 @@
    <link name="${prefix}front_left_wheel">
      <collision>
-       <origin xyz="0 0 0" rpy="0 0 0"/>
+       <origin xyz="0 0 0" rpy="${PI/2} 0 0"/>
        <geometry>
          <cylinder length="${wheel_width}" radius="${wheel_radius}"/>
@@ -42,5 +42,5 @@
      </collision>
      <visual>
-       <origin xyz="0 0 0" rpy="0 0 0"/>
+       <origin xyz="0 0 0" rpy="${PI/2} 0 0"/>
        <geometry>
          <cylinder length="${wheel_width}" radius="${wheel_radius}"/>
@@ -49,5 +49,5 @@
      </visual>
      <inertial>
-       <origin xyz="0 0 0" rpy="0 0 0"/>
+       <origin xyz="0 0 0" rpy="${PI/2} 0 0"/>
        <mass value="${wheel_mass}"/>
        <inertia

File: urdf/cmexamini/cmexamini_diff.ros2_control.xacro (robot description, xacro)
@@ -1,12 +1,12 @@
 <?xml version="1.0"?>
 <robot xmlns:xacro="http://www.ros.org/wiki/xacro">
-  <xacro:macro name="cmexb_ros2_control" params="name prefix use_mock_hardware">
+  <xacro:macro name="cmexamini_ros2_control" params="name prefix use_mock_hardware">
     <ros2_control name="${name}" type="system">
       <xacro:unless value="${use_mock_hardware}">
         <hardware>
-          <plugin>cmexa_base/CmexaMecanumBotSystemHardware</plugin>
-            <param name="example_param_hw_start_duration_sec">0</param>
-            <param name="example_param_hw_stop_duration_sec">3.0</param>
-            <param name="gear_ratio">5.0</param>
+          <plugin>cmexa_base/CmexaBaseBotSystemHardware</plugin>
+          <param name="example_param_hw_start_duration_sec">0</param>
+          <param name="example_param_hw_stop_duration_sec">3.0</param>
+          <param name="gear_ratio">1.0</param>
         </hardware>
         </xacro:unless>
