Commit message: test

File: urdf/cmexamini/cmexamini_properties.urdf.xacro (robot description, xacro)
@@ -4,8 +4,8 @@
   <!-- wheelbase = distance between wheel axis (x-direction)
        example: distance between wheel_front_right and wheel_rear_right-->
-  <xacro:property name="wheelbase" value="0.090" />
+  <xacro:property name="wheelbase" value="0.130" />
   <!-- track = distance between wheels (y-direction)
        example: distance between wheel_front_right and wheel_front_left -->
-  <xacro:property name="track" value="0.112" />
+  <xacro:property name="track" value="0.150"/>
   <!-- vertical offset means height -->
   <xacro:property name="wheel_vertical_offset" value="0.044" />
@@ -13,5 +13,5 @@
   <xacro:property name="wheel_radius" value="0.035" />
   <xacro:property name="wheel_width" value="0.015" />
-  <xacro:property name="gear_ratio" value="5.0"/>
+  <xacro:property name="gear_ratio" value="1.0"/>
   <xacro:property name="chassis_length" value="0.200" />
   <xacro:property name="chassis_width" value="0.130" />
