Commit message: feat(cmexamini): fix xacro includes and add LD19 laser frame
The mini's robot.urdf.xacro pointed at cmexamini_description/_properties/
_diff.ros2_control filenames that do not exist on disk (actual files are
robot_*), so xacro expansion failed. Point the includes at the real files.

Add a single forward-facing base_laser frame (one LDLiDAR LD19) so the mini
can run SLAM/nav and feed the webapp map. Mount pose is a placeholder pending
on-robot confirmation.

File: urdf/cmexamini/robot.urdf.xacro (robot description, xacro)
@@ -6,11 +6,11 @@
   <xacro:arg name="use_mock_hardware" default="false" />
   <!-- Import robot description -->
-  <xacro:include filename="$(find cmeresearch_description)/urdf/cmexamini/cmexamini_description.urdf.xacro" />
+  <xacro:include filename="$(find cmeresearch_description)/urdf/cmexamini/robot_description.urdf.xacro" />
   <!-- Robot constants and properties -->
-  <xacro:include filename="$(find cmeresearch_description)/urdf/cmexamini/cmexamini_properties.urdf.xacro" />
+  <xacro:include filename="$(find cmeresearch_description)/urdf/cmexamini/robot_properties.urdf.xacro" />
   <!-- Import Rviz colors -->
   <xacro:include filename="$(find cmeresearch_description)/urdf/materials.xacro" />
   <!-- Import ros2_control description -->
-  <xacro:include filename="$(find cmeresearch_description)/urdf/cmexamini/cmexamini_diff.ros2_control.xacro" />
+  <xacro:include filename="$(find cmeresearch_description)/urdf/cmexamini/robot_diff.ros2_control.xacro" />
   <!-- Instantiate the robot -->
   <xacro:cmexb prefix="$(arg prefix)" />

File: urdf/cmexamini/robot_description.urdf.xacro (robot description, xacro)
@@ -209,4 +209,38 @@
     </inertial>
   </link>
+  <!-- LiDAR (single LDLiDAR LD19). Unlike the mecanum cmexaiii (dual laser +
+       merger), the mini carries ONE forward-facing LD19 publishing directly on
+       /scan in frame base_laser. -->
+  <!-- TODO(on-robot): confirm the real mount pose. Placeholder mounts the LD19
+       front-centre, 0.12 m up. Adjust origin xyz/rpy to the physical mount and
+       the LD19 zero-heading before mapping. -->
+  <joint name="${prefix}base_laser_joint" type="fixed">
+    <origin xyz="0.05 0 0.12" rpy="0 0 0" />
+    <parent link="${prefix}base_link"/>
+    <child link="${prefix}base_laser" />
+  </joint>
+  <link name="${prefix}base_laser">
+    <collision>
+      <origin xyz="0 0 0" rpy="0 0 0"/>
+      <geometry>
+        <cylinder length="0.04" radius="0.02"/>
+      </geometry>
+    </collision>
+    <visual>
+      <origin xyz="0 0 0" rpy="0 0 0"/>
+      <geometry>
+        <cylinder length="0.04" radius="0.02"/>
+      </geometry>
+      <material name="orange"/>
+    </visual>
+    <inertial>
+      <origin xyz="0 0 0" rpy="0 0 0"/>
+      <mass value="0.2"/>
+      <inertia
+              ixx="0.0001" ixy="0.0" ixz="0.0"
+              iyy="0.0001" iyz="0.0"
+              izz="0.0001"/>
+    </inertial>
+  </link>
  </xacro:macro>
 </robot>
