Commit message: Renamed `cmexaiii_base` macro to `cmexaiii` in URDF Xacro for naming consistency.

File: urdf/cmexaiii/robot_description.urdf.xacro (robot description, xacro)
@@ -1,5 +1,5 @@
 <?xml version="1.0"?>
 <robot xmlns:xacro="http://www.ros.org/wiki/xacro">
-  <xacro:macro name="cmexaiii_base">
+  <xacro:macro name="cmexaiii">
   <xacro:property name="z_offset" value="-${chassis_height/2}" /> <!-- Space btw top of beam and the each joint -->
   <xacro:property name="wheel_mass" value="0.3"/>
