Commit message: Removed prefix usage from `cmexaiii` Xacro macros, standardized joint and link naming, updated related configurations, and renamed launch files for consistency.

File: urdf/cmexaiii/robot.urdf.xacro (robot description, xacro)
@@ -3,5 +3,4 @@
 <robot xmlns:xacro="http://www.ros.org/wiki/xacro" name="mecanumdrive_robot">
     <xacro:arg name="use_mock_hardware" default="false" />
-    <xacro:arg name="prefix" default="cmexaiii" />
     <!-- Robot constants and properties -->
     <xacro:include filename="$(find cmeresearch_description)/urdf/cmexaiii/robot_properties.urdf.xacro" />
@@ -13,6 +12,6 @@
     <xacro:include filename="$(find cmeresearch_description)/urdf/cmexaiii/robot_mecanum.ros2_control.xacro" />
     <!-- Instantiate the robot -->
-    <xacro:cmexaiii prefix="$(arg prefix)"/>
+    <xacro:cmexaiii_base />
     <!-- Add ros2_control -->
-    <xacro:cmexaiii_ros2_control name="CMEXAIII" prefix="$(arg prefix)" use_mock_hardware="$(arg use_mock_hardware)"/>
+    <xacro:cmexaiii_ros2_control name="CMEXAIII" use_mock_hardware="$(arg use_mock_hardware)"/>
 </robot>

File: urdf/cmexaiii/robot_description.urdf.xacro (robot description, xacro)
@@ -1,16 +1,16 @@
 <?xml version="1.0"?>
 <robot xmlns:xacro="http://www.ros.org/wiki/xacro">
-  <xacro:macro name="cmexaiii" params="prefix">
+  <xacro:macro name="cmexaiii_base">
   <xacro:property name="z_offset" value="-${chassis_height/2}" /> <!-- Space btw top of beam and the each joint -->
   <xacro:property name="wheel_mass" value="0.3"/>
   <!-- Base Link -->
-  <link name="${prefix}base_link">
+  <link name="base_link">
   </link>
-  <joint name="${prefix}base_link_joint" type="fixed">
+  <joint name="base_link_joint" type="fixed">
     <origin xyz="0 0 ${wheel_radius/2}" rpy="0 0 0" />
-    <parent link="${prefix}base_link"/>
-    <child link="${prefix}chassis_link" />
+    <parent link="base_link"/>
+    <child link="chassis_link" />
   </joint>
-  <link name="${prefix}chassis_link">
+  <link name="chassis_link">
     <visual>
       <origin xyz="${chassis_length/2} ${-chassis_width/2} 0" rpy="0 0 ${PI/2}" />
@@ -38,7 +38,7 @@
   </link>
     <!-- Front left wheel -->
-    <joint name="${prefix}front_left_wheel_joint" type="continuous">
-      <parent link="${prefix}base_link"/>
-      <child link="${prefix}front_left_wheel"/>
+    <joint name="front_left_wheel_joint" type="continuous">
+      <parent link="base_link"/>
+      <child link="front_left_wheel"/>
       <origin xyz="${wheelbase/2} ${track/2} ${wheel_radius/2}" rpy="0 0 0"/>
       <axis xyz="0 1 0"/>
@@ -47,5 +47,5 @@
     </joint>
     <!-- front left wheel Link -->
-    <link name="${prefix}front_left_wheel">
+    <link name="front_left_wheel">
       <collision>
         <origin xyz="0 0 0" rpy="${PI/2} 0 0"/>
@@ -71,7 +71,7 @@
     </link>
     <!-- Front right wheel -->
-    <joint name="${prefix}front_right_wheel_joint" type="continuous">
-      <parent link="${prefix}base_link"/>
-      <child link="${prefix}front_right_wheel"/>
+    <joint name="front_right_wheel_joint" type="continuous">
+      <parent link="base_link"/>
+      <child link="front_right_wheel"/>
       <origin xyz="${-wheelbase/2} ${track/2} ${wheel_radius/2}" rpy="0 0 0"/>
       <axis xyz="0 1 0"/>
@@ -80,5 +80,5 @@
     </joint>
     <!-- front right wheel Link -->
-    <link name="${prefix}front_right_wheel">
+    <link name="front_right_wheel">
       <collision>
         <origin xyz="0 0 0" rpy="${PI/2} 0 0"/>
@@ -104,7 +104,7 @@
     </link>
     <!-- rear left wheel -->
-    <joint name="${prefix}rear_left_wheel_joint" type="continuous">
-      <parent link="${prefix}base_link"/>
-      <child link="${prefix}rear_left_wheel"/>
+    <joint name="rear_left_wheel_joint" type="continuous">
+      <parent link="base_link"/>
+      <child link="rear_left_wheel"/>
       <origin xyz="${wheelbase/2} ${-track/2} ${wheel_radius/2}" rpy="0 0 0"/>
       <axis xyz="0 1 0"/>
@@ -113,5 +113,5 @@
     </joint>
     <!-- rear left wheel Link -->
-    <link name="${prefix}rear_left_wheel">
+    <link name="rear_left_wheel">
       <collision>
         <origin xyz="0 0 0" rpy="${PI/2} 0 0"/>
@@ -137,7 +137,7 @@
     </link>
     <!-- rear right wheel -->
-    <joint name="${prefix}rear_right_wheel_joint" type="continuous">
-      <parent link="${prefix}base_link"/>
-      <child link="${prefix}rear_right_wheel"/>
+    <joint name="rear_right_wheel_joint" type="continuous">
+      <parent link="base_link"/>
+      <child link="rear_right_wheel"/>
       <origin xyz="${-wheelbase/2} ${-track/2} ${wheel_radius/2}" rpy="0 0 0"/>
       <axis xyz="0 1 0"/>
@@ -146,5 +146,5 @@
     </joint>
     <!-- rear right wheel Link -->
-    <link name="${prefix}rear_right_wheel">
+    <link name="rear_right_wheel">
       <collision>
         <origin xyz="0 0 0" rpy="${PI/2} 0 0"/>
@@ -170,11 +170,11 @@
     </link>
     <!-- base_laser_front_joint -->
-    <joint name="${prefix}base_laser_front_joint" type="fixed">
+    <joint name="base_laser_front_joint" type="fixed">
       <origin xyz="0.460 0.257 0.18" rpy="0 0 -0.785" />
-      <parent link="${prefix}base_link"/>
-      <child link="${prefix}base_laser_front_left" />
+      <parent link="base_link"/>
+      <child link="base_laser_front_left" />
     </joint>
     <!-- front left laser Link -->
-    <link name="${prefix}base_laser_front_left">
+    <link name="base_laser_front_left">
       <collision>
         <origin xyz="0 0 0" rpy="0 0 0"/>
@@ -200,11 +200,11 @@
     </link>
     <!-- base_laser_rear_joint -->
-    <joint name="${prefix}base_laser_rear_joint" type="fixed">
+    <joint name="base_laser_rear_joint" type="fixed">
       <origin xyz="-0.460 -0.257 0.18" rpy="0 0 2.3562" />
-      <parent link="${prefix}base_link"/>
-      <child link="${prefix}base_laser_rear_right" />
+      <parent link="base_link"/>
+      <child link="base_laser_rear_right" />
     </joint>
     <!-- front left laser Link -->
-    <link name="${prefix}base_laser_rear_right">
+    <link name="base_laser_rear_right">
       <collision>
         <origin xyz="0 0 0" rpy="0 0 0"/>

File: urdf/cmexaiii/robot_mecanum.ros2_control.xacro (robot description, xacro)
@@ -1,5 +1,5 @@
 <?xml version="1.0"?>
 <robot xmlns:xacro="http://www.ros.org/wiki/xacro">
-    <xacro:macro name="cmexaiii_ros2_control" params="name prefix use_mock_hardware">
+    <xacro:macro name="cmexaiii_ros2_control" params="name use_mock_hardware">
         <ros2_control name="${name}" type="system">
             <xacro:unless value="${use_mock_hardware}">
@@ -21,20 +21,20 @@
                 </hardware>
             </xacro:if>
-            <joint name="${prefix}front_left_wheel_joint">
+            <joint name="front_left_wheel_joint">
                 <command_interface name="velocity"/>
                 <state_interface name="position"/>
                 <state_interface name="velocity"/>
             </joint>
-            <joint name="${prefix}rear_left_wheel_joint">
+            <joint name="rear_left_wheel_joint">
                 <command_interface name="velocity"/>
                 <state_interface name="position"/>
                 <state_interface name="velocity"/>
             </joint>
-            <joint name="${prefix}front_right_wheel_joint">
+            <joint name="front_right_wheel_joint">
                 <command_interface name="velocity"/>
                 <state_interface name="position"/>
                 <state_interface name="velocity"/>
             </joint>
-            <joint name="${prefix}rear_right_wheel_joint">
+            <joint name="rear_right_wheel_joint">
                 <command_interface name="velocity"/>
                 <state_interface name="position"/>

Commit message: Renamed `cmexaiii_base` to `cmexa_base` in URDF Xacro macros and updated related references for consistency.

File: urdf/cmexaiii/robot.urdf.xacro (robot description, xacro)
@@ -12,6 +12,6 @@
     <xacro:include filename="$(find cmeresearch_description)/urdf/cmexaiii/robot_mecanum.ros2_control.xacro" />
     <!-- Instantiate the robot -->
-    <xacro:cmexaiii_base />
+    <xacro:cmexa_base />
     <!-- Add ros2_control -->
-    <xacro:cmexaiii_ros2_control name="CMEXAIII" use_mock_hardware="$(arg use_mock_hardware)"/>
+    <xacro:cmexaiii_ros2_control name="cmexa_base" use_mock_hardware="$(arg use_mock_hardware)"/>
 </robot>

File: urdf/cmexaiii/robot_description.urdf.xacro (robot description, xacro)
@@ -1,5 +1,5 @@
 <?xml version="1.0"?>
 <robot xmlns:xacro="http://www.ros.org/wiki/xacro">
-  <xacro:macro name="cmexaiii_base">
+  <xacro:macro name="cmexa_base">
   <xacro:property name="z_offset" value="-${chassis_height/2}" /> <!-- Space btw top of beam and the each joint -->
   <xacro:property name="wheel_mass" value="0.3"/>

Commit message: Reverted `cmexa_base` to `cmexaiii_base` in URDF Xacro macros and updated related references for consistency.

File: urdf/cmexaiii/robot.urdf.xacro (robot description, xacro)
@@ -12,6 +12,6 @@
     <xacro:include filename="$(find cmeresearch_description)/urdf/cmexaiii/robot_mecanum.ros2_control.xacro" />
     <!-- Instantiate the robot -->
-    <xacro:cmexa_base />
+    <xacro:cmexaiii />
     <!-- Add ros2_control -->
-    <xacro:cmexaiii_ros2_control name="cmexa_base" use_mock_hardware="$(arg use_mock_hardware)"/>
+    <xacro:cmexaiii_ros2_control name="cmexaiii_base" use_mock_hardware="$(arg use_mock_hardware)"/>
 </robot>

File: urdf/cmexaiii/robot_description.urdf.xacro (robot description, xacro)
@@ -1,5 +1,5 @@
 <?xml version="1.0"?>
 <robot xmlns:xacro="http://www.ros.org/wiki/xacro">
-  <xacro:macro name="cmexa_base">
+  <xacro:macro name="cmexaiii_base">
   <xacro:property name="z_offset" value="-${chassis_height/2}" /> <!-- Space btw top of beam and the each joint -->
   <xacro:property name="wheel_mass" value="0.3"/>

Commit message: Added optional `prefix` parameter to `cmexaiii` and `cmexaiii_ros2_control` Xacro macros and updated related URDF and launch files for improved naming flexibility.

File: urdf/cmexaiii/robot.urdf.xacro (robot description, xacro)
@@ -3,4 +3,5 @@
 <robot xmlns:xacro="http://www.ros.org/wiki/xacro" name="mecanumdrive_robot">
     <xacro:arg name="use_mock_hardware" default="false" />
+    <xacro:arg name="prefix" default="" />
     <!-- Robot constants and properties -->
     <xacro:include filename="$(find cmeresearch_description)/urdf/cmexaiii/robot_properties.urdf.xacro" />
@@ -12,6 +13,6 @@
     <xacro:include filename="$(find cmeresearch_description)/urdf/cmexaiii/robot_mecanum.ros2_control.xacro" />
     <!-- Instantiate the robot -->
-    <xacro:cmexaiii />
+    <xacro:cmexaiii prefix="$(arg prefix)" />
     <!-- Add ros2_control -->
-    <xacro:cmexaiii_ros2_control name="cmexaiii_base" use_mock_hardware="$(arg use_mock_hardware)"/>
+    <xacro:cmexaiii_ros2_control name="cmexaiii" use_mock_hardware="$(arg use_mock_hardware)" prefix="$(arg prefix)"/>
 </robot>

File: urdf/cmexaiii/robot_mecanum.ros2_control.xacro (robot description, xacro)
@@ -1,5 +1,5 @@
 <?xml version="1.0"?>
 <robot xmlns:xacro="http://www.ros.org/wiki/xacro">
-    <xacro:macro name="cmexaiii_ros2_control" params="name use_mock_hardware">
+    <xacro:macro name="cmexaiii_ros2_control" params="name use_mock_hardware prefix">
         <ros2_control name="${name}" type="system">
             <xacro:unless value="${use_mock_hardware}">
@@ -21,20 +21,20 @@
                 </hardware>
             </xacro:if>
-            <joint name="front_left_wheel_joint">
+            <joint name="${prefix}front_left_wheel_joint">
                 <command_interface name="velocity"/>
                 <state_interface name="position"/>
                 <state_interface name="velocity"/>
             </joint>
-            <joint name="rear_left_wheel_joint">
+            <joint name="${prefix}rear_left_wheel_joint">
                 <command_interface name="velocity"/>
                 <state_interface name="position"/>
                 <state_interface name="velocity"/>
             </joint>
-            <joint name="front_right_wheel_joint">
+            <joint name="${prefix}front_right_wheel_joint">
                 <command_interface name="velocity"/>
                 <state_interface name="position"/>
                 <state_interface name="velocity"/>
             </joint>
-            <joint name="rear_right_wheel_joint">
+            <joint name="${prefix}rear_right_wheel_joint">
                 <command_interface name="velocity"/>
                 <state_interface name="position"/>
