Commit message: feat(cmexaiii): pass max_step_vel to cmexa_base for wheel normalization
cmexa_base now proportionally normalizes the four mecanum wheel commands
against a per-wheel ceiling derived from max_step_vel. Wire that parameter
through the cmexaiii ros2_control hardware block and define it in
robot_properties (8000 microsteps/s, matching the max_step_vel handed to
cmeresearch_stepper_driver in cmexaiii_hardware.launch.py).

Decoupled from the cmexa_base change: older cmexa_base ignores the extra
param, and a cmexa_base that supports it simply leaves normalization
disabled until this lands. Keep the two values in sync with the launch file.

File: urdf/cmexaiii/robot_mecanum.ros2_control.xacro (robot description, xacro)
@@ -14,4 +14,5 @@
                     <param name="steps_per_revolution">${steps_per_revolution}</param>
                     <param name="step_resolution">${step_resolution}</param>
+                    <param name="max_step_vel">${max_step_vel}</param>
                 </hardware>
             </xacro:unless>

File: urdf/cmexaiii/robot_properties.urdf.xacro (robot description, xacro)
@@ -13,4 +13,11 @@
        configured in cmeresearch_stepper_driver. 8 = 1/8 step (8 microsteps per full step). -->
   <xacro:property name="step_resolution" value="8" />
+  <!-- Per-wheel velocity ceiling in microsteps/s on the motor shaft. MUST match
+       the max_step_vel passed to cmeresearch_stepper_driver (see
+       cmexaiii_hardware.launch.py, currently 8000). cmexa_base uses this to
+       proportionally normalize the four mecanum wheel commands so combined
+       translation/rotation never over-drives two wheels while preserving the
+       commanded motion direction. -->
+  <xacro:property name="max_step_vel" value="8000" />
   <!-- vertical offset means height -->
   <xacro:property name="wheel_vertical_offset" value="0.01" />
